Commit message: Improve readability

File: cafe_robot_action_planning/robot_description/urdf/cafe_robot.urdf.xacro (robot description, xacro)
@@ -1,4 +1,7 @@
 <?xml version="1.0"?>
 <robot name="cafe_robot" xmlns:xacro="http://www.ros.org/wiki/xacro">
+    <xacro:include filename="inertial_macros.xacro"/>
+    <xacro:include filename="gazebo_plugins.xacro"/>
+    <xacro:include filename="inertial_macros.xacro"/>
     <!--                Dimensions              -->
     <xacro:property name="chassis_length" value="0.45"/>
@@ -12,32 +15,4 @@
     <xacro:property name="support_radius" value="0.01"/>
     <xacro:property name="support_pos_z" value="0.425"/>
-    <!--                Macro for Defining Inertia                  -->
-    <xacro:macro name="sphere_inertia" params="mass radius *origin">
-        <inertial>
-            <xacro:insert_block name="origin"/>
-            <mass value="${mass}" />
-            <inertia ixx="${(2/5) * mass * (radius*radius)}" ixy="0.0" ixz="0.0"
-                    iyy="${(2/5) * mass * (radius*radius)}" iyz="0.0"
-                    izz="${(2/5) * mass * (radius*radius)}" />
-        </inertial>
-    </xacro:macro>
-    <xacro:macro name="box_inertia" params="mass x y z *origin">
-        <inertial>
-            <xacro:insert_block name="origin"/>
-            <mass value="${mass}" />
-            <inertia ixx="${(1/12) * mass * (y*y+z*z)}" ixy="0.0" ixz="0.0"
-                    iyy="${(1/12) * mass * (x*x+z*z)}" iyz="0.0"
-                    izz="${(1/12) * mass * (x*x+y*y)}" />
-        </inertial>
-    </xacro:macro>
-    <xacro:macro name="cylinder_inertia" params="mass length radius *origin">
-        <inertial>
-            <xacro:insert_block name="origin"/>
-            <mass value="${mass}" />
-            <inertia ixx="${(1/12) * mass * (3*radius*radius + length*length)}" ixy="0.0" ixz="0.0"
-                    iyy="${(1/12) * mass * (3*radius*radius + length*length)}" iyz="0.0"
-                    izz="${(1/2) * mass * (radius*radius)}" />
-        </inertial>
-    </xacro:macro>
     <!--                Base Link               -->
     <link name="base_link"/>
@@ -56,9 +31,7 @@
     </joint>
     <link name="chassis_link">
-        <inertial>
-            <xacro:box_inertia mass="2.5" x="${chassis_length}" y="${chassis_width}" z="${chassis_height}">
-                <origin xyz="0 0 0" rpy="0 0 0"/>
-            </xacro:box_inertia>
-        </inertial>
+        <xacro:box_inertia mass="2.5" x="${chassis_length}" y="${chassis_width}" z="${chassis_height}">
+            <origin xyz="0 0 0" rpy="0 0 0"/>
+        </xacro:box_inertia>
         <visual>
             <origin xyz="0.0 0.0 0.0" rpy="0.0 0.0 0.0"/>
@@ -85,9 +58,7 @@
     </joint>
     <link name="wheel_L_link">
-        <inertial>
-            <xacro:cylinder_inertia mass="1.0" length="${wheel_thk}" radius="${wheel_radius}">
-                <origin xyz="0 0 0" rpy="0 0 0"/>
-            </xacro:cylinder_inertia>
-        </inertial>
+        <xacro:cylinder_inertia mass="1.0" length="${wheel_thk}" radius="${wheel_radius}">
+            <origin xyz="0 0 0" rpy="0 0 0"/>
+        </xacro:cylinder_inertia>
         <visual>
             <origin xyz="0.0 0.0 0.0" rpy=" 0.0 0.0 0.0"/>
@@ -114,9 +85,7 @@
     </joint>
     <link name="wheel_R_link">
-        <inertial>
-            <xacro:cylinder_inertia mass="1.0" length="${wheel_thk}" radius="${wheel_radius}">
-                <origin xyz="0 0 0" rpy="0 0 0"/>
-            </xacro:cylinder_inertia>
-        </inertial>
+        <xacro:cylinder_inertia mass="1.0" length="${wheel_thk}" radius="${wheel_radius}">
+            <origin xyz="0 0 0" rpy="0 0 0"/>
+        </xacro:cylinder_inertia>
         <visual>
             <origin xyz="0.0 0.0 0.0" rpy="0.0 0.0 0.0"/>
@@ -142,9 +111,7 @@
     </joint>
     <link name="caster_wheelF">
-        <inertial>
-            <xacro:sphere_inertia mass="0.15" radius="0.03">
-                <origin xyz="0 0 0" rpy="0 0 0"/>
-            </xacro:sphere_inertia>
-        </inertial>
+        <xacro:sphere_inertia mass="0.15" radius="0.03">
+            <origin xyz="0 0 0" rpy="0 0 0"/>
+        </xacro:sphere_inertia>
         <visual>
             <origin xyz="0.0 0.0 0.0" rpy=" 0.0 0.0 0.0"/>
@@ -169,9 +136,7 @@
     </joint>
     <link name="caster_wheelB">
-        <inertial>
-            <xacro:sphere_inertia mass="0.15" radius="0.03">
-                <origin xyz="0 0 0" rpy="0 0 0"/>
-            </xacro:sphere_inertia>
-        </inertial>
+        <xacro:sphere_inertia mass="0.15" radius="0.03">
+            <origin xyz="0 0 0" rpy="0 0 0"/>
+        </xacro:sphere_inertia>
         <visual>
             <origin xyz="0.0 0.0 0.0" rpy=" 0.0 0.0 0.0"/>
@@ -197,9 +162,7 @@
     </joint>
     <link name="lidar_frame">
-        <inertial>
-            <xacro:cylinder_inertia mass="0.200" length="${lidar_height}" radius="${lidar_radius}">
-                <origin xyz="0 0 0" rpy="0 0 0"/>
-            </xacro:cylinder_inertia>
-        </inertial>
+        <xacro:cylinder_inertia mass="0.200" length="${lidar_height}" radius="${lidar_radius}">
+            <origin xyz="0 0 0" rpy="0 0 0"/>
+        </xacro:cylinder_inertia>
         <visual>
             <origin xyz="0.0 0.0 0.0" rpy=" 0.0 0.0 0.0"/>
@@ -225,9 +188,7 @@
     </joint>
     <link name="support1">
-        <inertial>
-            <xacro:cylinder_inertia mass="0.3" length="${support_height}" radius="${support_radius}">
-                <origin xyz="0 0 0" rpy="0 0 0"/>
-            </xacro:cylinder_inertia>
-        </inertial>
+        <xacro:cylinder_inertia mass="0.3" length="${support_height}" radius="${support_radius}">
+            <origin xyz="0 0 0" rpy="0 0 0"/>
+        </xacro:cylinder_inertia>
         <visual>
             <origin xyz="0.0 0.0 0.0" rpy="0.0 0.0 0.0"/>
@@ -253,9 +214,7 @@
     </joint>
     <link name="support2">
-        <inertial>
-            <xacro:cylinder_inertia mass="0.3" length="${support_height}" radius="${support_radius}">
-                <origin xyz="0 0 0" rpy="0 0 0"/>
-            </xacro:cylinder_inertia>
-        </inertial>
+        <xacro:cylinder_inertia mass="0.3" length="${support_height}" radius="${support_radius}">
+            <origin xyz="0 0 0" rpy="0 0 0"/>
+        </xacro:cylinder_inertia>
         <visual>
             <origin xyz="0.0 0.0 0.0" rpy="0.0 0.0 0.0"/>
@@ -281,9 +240,7 @@
     </joint>
     <link name="support3">
-        <inertial>
-            <xacro:cylinder_inertia mass="0.3" length="${support_height}" radius="${support_radius}">
-                <origin xyz="0 0 0" rpy="0 0 0"/>
-            </xacro:cylinder_inertia>
-        </inertial>
+        <xacro:cylinder_inertia mass="0.3" length="${support_height}" radius="${support_radius}">
+            <origin xyz="0 0 0" rpy="0 0 0"/>
+        </xacro:cylinder_inertia>
         <visual>
             <origin xyz="0.0 0.0 0.0" rpy="0.0 0.0 0.0"/>
@@ -309,9 +266,7 @@
     </joint>
     <link name="support4">
-        <inertial>
-            <xacro:cylinder_inertia mass="0.3" length="${support_height}" radius="${support_radius}">
-                <origin xyz="0 0 0" rpy="0 0 0"/>
-            </xacro:cylinder_inertia>
-        </inertial>
+        <xacro:cylinder_inertia mass="0.3" length="${support_height}" radius="${support_radius}">
+            <origin xyz="0 0 0" rpy="0 0 0"/>
+        </xacro:cylinder_inertia>
         <visual>
             <origin xyz="0.0 0.0 0.0" rpy="0.0 0.0 0.0"/>
@@ -338,9 +293,7 @@
     </joint>
     <link name="level1">
-        <inertial>
-            <xacro:cylinder_inertia mass="0.3" length="${wheel_thk}" radius="${wheel_radius}">
-                <origin xyz="0 0 0" rpy="0 0 0"/>
-            </xacro:cylinder_inertia>
-        </inertial>
+        <xacro:cylinder_inertia mass="0.3" length="${wheel_thk}" radius="${wheel_radius}">
+            <origin xyz="0 0 0" rpy="0 0 0"/>
+        </xacro:cylinder_inertia>
         <visual>
             <origin xyz="0.0 0.0 0.0" rpy="0.0 0.0 0.0"/>
@@ -365,9 +318,7 @@
     </joint>
     <link name="level2">
-        <inertial>
-            <xacro:cylinder_inertia mass="0.3" length="${wheel_thk}" radius="${wheel_radius}">
-                <origin xyz="0 0 0" rpy="0 0 0"/>
-            </xacro:cylinder_inertia>
-        </inertial>
+        <xacro:cylinder_inertia mass="0.3" length="${wheel_thk}" radius="${wheel_radius}">
+            <origin xyz="0 0 0" rpy="0 0 0"/>
+        </xacro:cylinder_inertia>
         <visual>
             <origin xyz="0.0 0.0 0.0" rpy="0.0 0.0 0.0"/>
@@ -392,9 +343,7 @@
     </joint>
     <link name="level3">
-        <inertial>
-            <xacro:cylinder_inertia mass="0.3" length="${wheel_thk}" radius="${wheel_radius}">
-                <origin xyz="0 0 0" rpy="0 0 0"/>
-            </xacro:cylinder_inertia>
-        </inertial>
+        <xacro:cylinder_inertia mass="0.3" length="${wheel_thk}" radius="${wheel_radius}">
+            <origin xyz="0 0 0" rpy="0 0 0"/>
+        </xacro:cylinder_inertia>
         <visual>
             <origin xyz="0.0 0.0 0.0" rpy="0.0 0.0 0.0"/>
@@ -413,51 +362,3 @@
         </collision>
     </link>
-    <!--                Gazebo Plugins              -->
-    <gazebo reference="lidar_frame">
-        <sensor name="laser" type="gpu_lidar">
-            <pose> 0 0 0 0 0 0 </pose>
-            <visualize>false</visualize>
-            <update_rate>10</update_rate>
-            <lidar>
-                <scan>
-                    <horizontal>
-                        <samples>360</samples>
-                        <min_angle>-3.14</min_angle>
-                        <max_angle>3.14</max_angle>
-                    </horizontal>
-                </scan>
-                <range>
-                    <min>0.3</min>
-                    <max>12</max>
-                </range>
-            </lidar>
-            <topic>scan</topic>
-            <gz_frame_id>laser_frame</gz_frame_id>
-        </sensor>
-    </gazebo>
-    <gazebo>
-        <plugin name="gz::sim::systems::DiffDrive" filename="gz-sim-diff-drive-system">
-            <!-- Wheel Info -->
-            <left_joint>wheel_L_joint</left_joint>
-            <right_joint>wheel_R_joint</right_joint>
-            <wheel_separation>${chassis_width + wheel_thk}</wheel_separation>
-            <wheel_radius>${wheel_radius}</wheel_radius>
-            <!-- Limits -->
-            <max_linear_acceleration>0.33</max_linear_acceleration>
-            <!-- Input -->
-            <topic>cmd_vel</topic>
-            <!-- Output -->
-            <frame_id>odom</frame_id>
-            <child_frame_id>base_link</child_frame_id>
-            <odom_topic>odom</odom_topic>
-            <odom_publisher_frequency>30</odom_publisher_frequency>
-            <tf_topic>/tf</tf_topic>
-        </plugin>
-        <plugin filename="gz-sim-joint-state-publisher-system"
-            name="gz::sim::systems::JointStatePublisher">
-            <topic>joint_states</topic>
-            <joint_name>wheel_L_joint</joint_name>
-            <joint_name>wheel_R_joint</joint_name>
-        </plugin>
-    </gazebo>
 </robot>

Commit message: Change position caster_wheel link

File: cafe_robot_action_planning/robot_description/urdf/cafe_robot.urdf.xacro (robot description, xacro)
@@ -55,5 +55,5 @@
         <child link="wheel_L_link"/>
         <axis xyz="0 0 1"/>
-        <origin xyz="0 0.225 -0.04" rpy="1.57 0 0"/>
+        <origin xyz="0 0.225 -0.03" rpy="1.57 0 0"/>
     </joint>
     <link name="wheel_L_link">
@@ -82,5 +82,5 @@
         <child link="wheel_R_link"/>
         <axis xyz="0 0 1"/>
-        <origin xyz="0 -0.225 -0.04" rpy="1.57 0 0"/>
+        <origin xyz="0 -0.225 -0.03" rpy="1.57 0 0"/>
     </joint>
     <link name="wheel_R_link">
@@ -130,4 +130,9 @@
         </collision>
     </link>
+    <gazebo reference="caster_wheelF">
+        <material>Gazebo/White</material>
+        <mu1 value="0.001"/>
+        <mu2 value="0.001"/>
+    </gazebo>
     <joint name="caster_wheelB_joint" type="fixed">
         <parent link="base_link"/>
@@ -155,4 +160,9 @@
         </collision>
     </link>
+    <gazebo reference="caster_wheelB">
+        <material>Gazebo/White</material>
+        <mu1 value="0.001"/>
+        <mu2 value="0.001"/>
+    </gazebo>
     <!--                Laser joint & link              -->
     <joint name="lidar_joint" type="fixed">

Commit message: Change Wheels & gazebo plugin

File: cafe_robot_action_planning/robot_description/urdf/cafe_robot.urdf.xacro (robot description, xacro)
@@ -50,8 +50,8 @@
         </collision>
     </link>
-    <!--            Left Wheel Joint                -->
-    <joint name="wheel_L_joint" type="continuous">
-        <parent link="base_link"/>
-        <child link="wheel_L_link"/>
+    <!--            Right Wheel Joint                -->
+    <joint name="wheel_R_joint" type="continuous">
+        <parent link="base_link"/>
+        <child link="wheel_R_link"/>
         <axis xyz="0 0 1"/>
         <origin xyz="0 0.225 -0.03" rpy="1.57 0 0"/>
@@ -77,8 +77,8 @@
         </collision>
     </link>
-    <!--                Right Wheel Joint               -->
-    <joint name="wheel_R_joint" type="continuous">
-        <parent link="base_link"/>
-        <child link="wheel_R_link"/>
+    <!--                Left Wheel Joint               -->
+    <joint name="wheel_L_joint" type="continuous">
+        <parent link="base_link"/>
+        <child link="wheel_L_link"/>
         <axis xyz="0 0 1"/>
         <origin xyz="0 -0.225 -0.03" rpy="1.57 0 0"/>
@@ -168,5 +168,5 @@
     <joint name="lidar_joint" type="fixed">
         <parent link="base_link"/>
-        <child link="lidar_frame"/>
+        <child link="laser_frame"/>
         <origin xyz="0 0 0.125" rpy="0.0 0 0"/>
     </joint>

File: cafe_robot_action_planning/robot_description/urdf/gazebo_plugins.xacro (robot description, xacro)
@@ -3,4 +3,5 @@
     <!--                Gazebo Plugins              -->
     <gazebo reference="lidar_frame">
+        <material>Gazebo/Black</material>
         <sensor name="laser" type="gpu_lidar">
             <pose> 0 0 0 0 0 0 </pose>
@@ -21,5 +22,5 @@
             </lidar>
             <topic>scan</topic>
-            <gz_frame_id>laser_frame</gz_frame_id>
+            <gz_frame_id>lidar_frame</gz_frame_id>
         </sensor>
     </gazebo>

Commit message: Fix LiDAR Visualization

File: cafe_robot_action_planning/robot_description/urdf/cafe_robot.urdf.xacro (robot description, xacro)
@@ -106,5 +106,5 @@
     <!--                Caster wheel joints & links              -->
     <joint name="caster_wheelF_joint" type="fixed">
-        <parent link="base_link"/>
+        <parent link="chassis_link"/>
         <child link="caster_wheelF"/>
         <origin xyz="0.15 0 -0.1" rpy="0.0 0 0"/>
@@ -136,5 +136,5 @@
     </gazebo>
     <joint name="caster_wheelB_joint" type="fixed">
-        <parent link="base_link"/>
+        <parent link="chassis_link"/>
         <child link="caster_wheelB"/>
         <origin xyz="-0.15 0 -0.1" rpy="0.0 0 0"/>
@@ -167,9 +167,9 @@
     <!--                Laser joint & link              -->
     <joint name="lidar_joint" type="fixed">
-        <parent link="base_link"/>
+        <parent link="chassis_link"/>
         <child link="laser_frame"/>
         <origin xyz="0 0 0.125" rpy="0.0 0 0"/>
     </joint>
-    <link name="lidar_frame">
+    <link name="laser_frame">
         <xacro:cylinder_inertia mass="0.200" length="${lidar_height}" radius="${lidar_radius}">
             <origin xyz="0 0 0" rpy="0 0 0"/>
@@ -193,5 +193,5 @@
     <!--            Support Frames              -->
     <joint name="support1_joint" type="fixed">
-        <parent link="base_link"/>
+        <parent link="chassis_link"/>
         <child link="support1"/>
         <origin xyz="0.18 0.15 ${support_pos_z}" rpy="0.0 0.0 0.0"/>
@@ -219,5 +219,5 @@
     </link>
     <joint name="support2_joint" type="fixed">
-        <parent link="base_link"/>
+        <parent link="chassis_link"/>
         <child link="support2"/>
         <origin xyz="-0.18 -0.15 ${support_pos_z}" rpy="0.0 0.0 0.0"/>
@@ -245,5 +245,5 @@
     </link>
     <joint name="support3_joint" type="fixed">
-        <parent link="base_link"/>
+        <parent link="chassis_link"/>
         <child link="support3"/>
         <origin xyz="-0.18 0.15 ${support_pos_z}" rpy="0.0 0.0 0.0"/>
@@ -271,5 +271,5 @@
     </link>
     <joint name="support4_joint" type="fixed">
-        <parent link="base_link"/>
+        <parent link="chassis_link"/>
         <child link="support4"/>
         <origin xyz="0.18 -0.15 ${support_pos_z}" rpy="0.0 0.0 0.0"/>
@@ -298,5 +298,5 @@
     <!--                Level Frames              -->
     <joint name="level1_joint" type="fixed">
-        <parent link="base_link"/>
+        <parent link="chassis_link"/>
         <child link="level1"/>
         <origin xyz="0 0 0.25" rpy="0.0 0.0 0.0"/>
@@ -323,5 +323,5 @@
     </link>
     <joint name="level2_joint" type="fixed">
-        <parent link="base_link"/>
+        <parent link="chassis_link"/>
         <child link="level2"/>
         <origin xyz="0 0 0.5" rpy="0.0 0.0 0.0"/>
@@ -348,5 +348,5 @@
     </link>
     <joint name="level3_joint" type="fixed">
-        <parent link="base_link"/>
+        <parent link="chassis_link"/>
         <child link="level3"/>
         <origin xyz="0 0 0.75" rpy="0.0 0.0 0.0"/>

File: cafe_robot_action_planning/robot_description/urdf/gazebo_plugins.xacro (robot description, xacro)
@@ -2,5 +2,5 @@
 <robot xmlns:xacro="http://www.ros.org/wiki/xacro" name="cafe_robot">
     <!--                Gazebo Plugins              -->
-    <gazebo reference="lidar_frame">
+    <gazebo reference="laser_frame">
         <material>Gazebo/Black</material>
         <sensor name="laser" type="gpu_lidar">
@@ -22,5 +22,5 @@
             </lidar>
             <topic>scan</topic>
-            <gz_frame_id>lidar_frame</gz_frame_id>
+            <gz_frame_id>laser_frame</gz_frame_id>
         </sensor>
     </gazebo>

Commit message: Fix wheel definitions

File: cafe_robot_action_planning/robot_description/urdf/cafe_robot.urdf.xacro (robot description, xacro)
@@ -50,40 +50,38 @@
         </collision>
     </link>
-    <!--            Right Wheel Joint                -->
-    <joint name="wheel_R_joint" type="continuous">
-        <parent link="base_link"/>
-        <child link="wheel_R_link"/>
-        <axis xyz="0 0 1"/>
-        <origin xyz="0 0.225 -0.03" rpy="1.57 0 0"/>
-    </joint>
-    <link name="wheel_L_link">
-        <xacro:cylinder_inertia mass="1.0" length="${wheel_thk}" radius="${wheel_radius}">
-            <origin xyz="0 0 0" rpy="0 0 0"/>
-        </xacro:cylinder_inertia>
-        <visual>
-            <origin xyz="0.0 0.0 0.0" rpy=" 0.0 0.0 0.0"/>
-            <geometry>
-                <cylinder radius="${wheel_radius}" length="${wheel_thk}"/>
-            </geometry>
-            <material name="grey">
-                <color rgba="0.1 0.7 0.7 1.0"/>
-            </material>
-        </visual>
-        <collision>
-            <origin xyz="0.0 0.0 0.0" rpy="0.0 0.0 0.0"/>
-            <geometry>
-                <cylinder radius="${wheel_radius}" length="${wheel_thk}"/>
-            </geometry>
-        </collision>
-    </link>
-    <!--                Left Wheel Joint               -->
     <joint name="wheel_L_joint" type="continuous">
+        <origin xyz="0 0.225 -0.03" rpy="-1.57 0.0 0.0"/>
         <parent link="base_link"/>
         <child link="wheel_L_link"/>
         <axis xyz="0 0 1"/>
-        <origin xyz="0 -0.225 -0.03" rpy="1.57 0 0"/>
+    </joint>
+    <link name="wheel_L_link">
+        <xacro:cylinder_inertia mass="0.3" length="${wheel_thk}" radius="${wheel_radius}">
+            <origin xyz="0 0 0" rpy="0 0 0"/>
+        </xacro:cylinder_inertia>
+        <visual>
+            <origin xyz="0.0 0.0 0.0" rpy="0.0 0.0 0.0"/>
+            <geometry>
+                <cylinder radius="${wheel_radius}" length="${wheel_thk}"/>
+            </geometry>
+            <material name="goat">
+                <color rgba="0.1 0.7 0.7 1.0"/>
+            </material>
+        </visual>
+        <collision>
+            <origin xyz="0.0 0.0 0.0" rpy="0.0 0.0 0.0"/>
+            <geometry>
+                <cylinder radius="${wheel_radius}" length="${wheel_thk}"/>
+            </geometry>
+        </collision>
+    </link>
+     <joint name="wheel_R_joint" type="continuous">
+        <origin xyz="0 -0.225 -0.03" rpy="1.57 0.0 0.0"/>
+        <parent link="base_link"/>
+        <child link="wheel_R_link"/>
+        <axis xyz="0 0 -1"/>
     </joint>
     <link name="wheel_R_link">
-        <xacro:cylinder_inertia mass="1.0" length="${wheel_thk}" radius="${wheel_radius}">
+        <xacro:cylinder_inertia mass="0.3" length="${wheel_thk}" radius="${wheel_radius}">
             <origin xyz="0 0 0" rpy="0 0 0"/>
         </xacro:cylinder_inertia>
@@ -93,5 +91,5 @@
                 <cylinder radius="${wheel_radius}" length="${wheel_thk}"/>
             </geometry>
-            <material name="grey">
+            <material name="goat">
                 <color rgba="0.1 0.7 0.7 1.0"/>
             </material>

Commit message: Add Simulation Env

File: cafe_robot_action_planning/robot_description/urdf/cafe_robot.urdf.xacro (robot description, xacro)
@@ -50,4 +50,5 @@
         </collision>
     </link>
+    <!--                Left Wheel Joint               -->
     <joint name="wheel_L_joint" type="continuous">
         <origin xyz="0 0.225 -0.03" rpy="-1.57 0.0 0.0"/>
@@ -76,4 +77,5 @@
         </collision>
     </link>
+     <!--           Right Wheel Joint              -->
      <joint name="wheel_R_joint" type="continuous">
         <origin xyz="0 -0.225 -0.03" rpy="1.57 0.0 0.0"/>
@@ -370,3 +372,28 @@
         </collision>
     </link>
+    <joint name="misc_joint" type="fixed">
+        <parent link="base_link"/>
+        <child link="misc_link"/>
+        <origin xyz="0.2 0.0 0.075" rpy="0.0 0.0 0.0"/>
+    </joint>
+     <link name="misc_link">
+        <xacro:sphere_inertia mass="0.05" radius="0.03">
+            <origin xyz="0 0 0" rpy="0 0 0"/>
+        </xacro:sphere_inertia>
+        <visual>
+            <origin xyz="0.0 0.0 0.0" rpy=" 0.0 0.0 0.0"/>
+            <geometry>
+                <sphere radius="0.03"/>
+            </geometry>
+            <material name="black">
+                <color rgba="0.0 0.0 0.0 1.0"/>
+            </material>
+        </visual>
+        <collision>
+            <origin xyz="0.0 0.0 0.0" rpy="0.0 0.0 0.0"/>
+            <geometry>
+                <sphere radius="0.03"/>
+            </geometry>
+        </collision>
+    </link>
 </robot>
